Commit message: Add URDF
Adds a basic robot description including a URDF, RViz config, and a launch file to publish the URDF.

The URDF defines the robot's base link and links for the DVL, USBL, FLS, and Voyis stereo cameras.

The RViz config provides a default visualization setup.

The launch file publishes the URDF to the /robot_description topic using the robot_state_publisher.

File: urdf/rhody.urdf.xacro (robot description, xacro)
@@ -3,8 +3,9 @@
   <xacro:arg name="namespace" default="rhody" />
   <xacro:property name="namespace" value="$(arg namespace)" scope="global" />
-  <xacro:property name="deg" value="${pi/180}" />
+  <xacro:property name="deg" value="${pi / 180.0}" />
+  <!-- Base Link -->
   <link name="${namespace}/base_link">
     <visual>
-      <origin rpy="0.0 0 0" xyz="0 0 0"/>
+      <origin xyz="0 0 0" rpy="0 0 0"/>
       <geometry>
         <mesh filename="package://rhody/meshes/rhody.dae"/>
@@ -12,3 +13,38 @@
     </visual>
   </link>
+  <!-- DVL Link -->
+  <link name="${namespace}/dvl_link"/>
+  <joint name="${namespace}_base_to_dvl" type="fixed">
+    <parent link="${namespace}/base_link"/>
+    <child link="${namespace}/dvl_link"/>
+    <origin xyz="0 0 0" rpy="0 0 0"/>
+  </joint>
+  <!-- USBL -->
+  <link name="${namespace}/usbl_link"/>
+  <joint name="${namespace}_base_to_usbl" type="fixed">
+    <parent link="${namespace}/base_link"/>
+    <child link="${namespace}/usbl_link"/>
+    <origin xyz="0.013 0.050 0.385" rpy="0 0 0"/>
+  </joint>
+  <!-- FLS -->
+  <link name="${namespace}/fls_link"/>
+  <joint name="${namespace}_base_to_fls" type="fixed">
+    <parent link="${namespace}/base_link"/>
+    <child link="${namespace}/fls_link"/>
+    <origin xyz="0.338 0.050 0.281" rpy="0 ${5.0 * deg} 0"/>
+  </joint>
+  <!-- Voyis Stereo: Left Entrance Pupil -->
+  <link name="${namespace}/voyis_left_link"/>
+  <joint name="${namespace}_base_to_voyis_left" type="fixed">
+    <parent link="${namespace}/base_link"/>
+    <child link="${namespace}/voyis_left_link"/>
+    <origin xyz="0.323 -0.035 -0.008" rpy="0 0 0"/>
+  </joint>
+  <!-- Voyis Stereo: Right Entrance Pupil -->
+  <link name="${namespace}/voyis_right_link"/>
+  <joint name="${namespace}_base_to_voyis_right" type="fixed">
+    <parent link="${namespace}/base_link"/>
+    <child link="${namespace}/voyis_right_link"/>
+    <origin xyz="0.323 0.135 -0.008" rpy="0 0 0"/>
+  </joint>
 </robot>

Commit message: removed namespacing from tf to simplify, changed config for testing
still not working, ekf exploding

File: urdf/rhody.urdf.xacro (robot description, xacro)
@@ -5,5 +5,5 @@
   <xacro:property name="deg" value="${pi / 180.0}" />
   <!-- Base Link -->
-  <link name="${namespace}/base_link">
+  <link name="base_link">
     <visual>
       <origin xyz="0 0 0" rpy="0 0 0"/>
@@ -14,36 +14,36 @@
   </link>
   <!-- DVL Link -->
-  <link name="${namespace}/dvl_link"/>
-  <joint name="${namespace}_base_to_dvl" type="fixed">
-    <parent link="${namespace}/base_link"/>
-    <child link="${namespace}/dvl_link"/>
+  <link name="dvl_link"/>
+  <joint name="base_to_dvl" type="fixed">
+    <parent link="base_link"/>
+    <child link="dvl_link"/>
     <origin xyz="0 0 0" rpy="0 0 0"/>
   </joint>
   <!-- USBL -->
-  <link name="${namespace}/usbl_link"/>
-  <joint name="${namespace}_base_to_usbl" type="fixed">
-    <parent link="${namespace}/base_link"/>
-    <child link="${namespace}/usbl_link"/>
+  <link name="usbl_link"/>
+  <joint name="base_to_usbl" type="fixed">
+    <parent link="base_link"/>
+    <child link="usbl_link"/>
     <origin xyz="0.013 0.050 0.385" rpy="0 0 0"/>
   </joint>
   <!-- FLS -->
-  <link name="${namespace}/fls_link"/>
-  <joint name="${namespace}_base_to_fls" type="fixed">
-    <parent link="${namespace}/base_link"/>
-    <child link="${namespace}/fls_link"/>
+  <link name="fls_link"/>
+  <joint name="base_to_fls" type="fixed">
+    <parent link="base_link"/>
+    <child link="fls_link"/>
     <origin xyz="0.338 0.050 0.281" rpy="0 ${5.0 * deg} 0"/>
   </joint>
   <!-- Voyis Stereo: Left Entrance Pupil -->
-  <link name="${namespace}/voyis_left_link"/>
-  <joint name="${namespace}_base_to_voyis_left" type="fixed">
-    <parent link="${namespace}/base_link"/>
-    <child link="${namespace}/voyis_left_link"/>
+  <link name="voyis_left_link"/>
+  <joint name="base_to_voyis_left" type="fixed">
+    <parent link="base_link"/>
+    <child link="voyis_left_link"/>
     <origin xyz="0.323 -0.035 -0.008" rpy="0 0 0"/>
   </joint>
   <!-- Voyis Stereo: Right Entrance Pupil -->
-  <link name="${namespace}/voyis_right_link"/>
-  <joint name="${namespace}_base_to_voyis_right" type="fixed">
-    <parent link="${namespace}/base_link"/>
-    <child link="${namespace}/voyis_right_link"/>
+  <link name="voyis_right_link"/>
+  <joint name="base_to_voyis_right" type="fixed">
+    <parent link="base_link"/>
+    <child link="voyis_right_link"/>
     <origin xyz="0.323 0.135 -0.008" rpy="0 0 0"/>
   </joint>
