Commit message: basic rhody urdf with optical and sonar frames

File: urdf/rhody.urdf.xacro (robot description, xacro)
@@ -4,4 +4,12 @@
   <xacro:property name="namespace" value="$(arg namespace)" scope="global" />
   <xacro:property name="deg" value="${pi / 180.0}" />
+  <!-- base_link follows REP-103: x forward, y port, z up.
+       The CAD offsets these links came from use y starboard, so all y values
+       below are negated with respect to the CAD numbers. -->
+  <!-- STL carries no color, so give the link an explicit material.
+       Without one RViz renders the mesh red. -->
+  <material name="rhody_grey">
+    <color rgba="0.75 0.75 0.78 1.0"/>
+  </material>
   <!-- Base Link -->
   <link name="base_link">
@@ -9,6 +17,8 @@
       <origin xyz="0 0 0" rpy="0 0 0"/>
       <geometry>
-        <mesh filename="package://rhody/meshes/rhody.dae"/>
+        <!-- Exported in meters, already x-forward / y-port / z-up -->
+        <mesh filename="package://rhody/meshes/JM00004388_decimated.STL"/>
       </geometry>
+      <material name="rhody_grey"/>
     </visual>
   </link>
@@ -25,5 +35,5 @@
     <parent link="base_link"/>
     <child link="usbl_link"/>
-    <origin xyz="0.013 0.050 0.385" rpy="0 0 0"/>
+    <origin xyz="0.013 -0.050 0.385" rpy="0 0 0"/>
   </joint>
   <!-- FLS -->
@@ -32,19 +42,30 @@
     <parent link="base_link"/>
     <child link="fls_link"/>
-    <origin xyz="0.338 0.050 0.281" rpy="0 ${5.0 * deg} 0"/>
+    <origin xyz="0.338 -0.050 0.281" rpy="0 ${5.0 * deg} 0"/>
   </joint>
-  <!-- Voyis Stereo: Left Entrance Pupil -->
+  <!-- Camera optical frame: z forward, x right, y down (REP-103 / ISAAC ROS) -->
+  <xacro:macro name="optical_frame" params="name parent">
+    <link name="${name}"/>
+    <joint name="${parent}_to_${name}" type="fixed">
+      <parent link="${parent}"/>
+      <child link="${name}"/>
+      <origin xyz="0 0 0" rpy="${-pi/2} 0 ${-pi/2}"/>
+    </joint>
+  </xacro:macro>
+  <!-- Voyis Stereo: Left Entrance Pupil (port side) -->
   <link name="voyis_left_link"/>
   <joint name="base_to_voyis_left" type="fixed">
     <parent link="base_link"/>
     <child link="voyis_left_link"/>
-    <origin xyz="0.323 -0.035 -0.008" rpy="0 0 0"/>
+    <origin xyz="0.323 0.035 -0.008" rpy="0 0 0"/>
   </joint>
-  <!-- Voyis Stereo: Right Entrance Pupil -->
+  <xacro:optical_frame name="voyis_left_optical_frame" parent="voyis_left_link"/>
+  <!-- Voyis Stereo: Right Entrance Pupil (starboard side) -->
   <link name="voyis_right_link"/>
   <joint name="base_to_voyis_right" type="fixed">
     <parent link="base_link"/>
     <child link="voyis_right_link"/>
-    <origin xyz="0.323 0.135 -0.008" rpy="0 0 0"/>
+    <origin xyz="0.323 -0.135 -0.008" rpy="0 0 0"/>
   </joint>
+  <xacro:optical_frame name="voyis_right_optical_frame" parent="voyis_right_link"/>
 </robot>

Commit message: voyis nvidia slam demo

File: urdf/rhody.urdf.xacro (robot description, xacro)
@@ -59,5 +59,5 @@
     <origin xyz="0.323 0.035 -0.008" rpy="0 0 0"/>
   </joint>
-  <xacro:optical_frame name="voyis_left_optical_frame" parent="voyis_left_link"/>
+  <xacro:optical_frame name="voyis_left_optical" parent="voyis_left_link"/>
   <!-- Voyis Stereo: Right Entrance Pupil (starboard side) -->
   <link name="voyis_right_link"/>
@@ -67,4 +67,14 @@
     <origin xyz="0.323 -0.135 -0.008" rpy="0 0 0"/>
   </joint>
-  <xacro:optical_frame name="voyis_right_optical_frame" parent="voyis_right_link"/>
+  <xacro:optical_frame name="voyis_right_optical" parent="voyis_right_link"/>
+  <!-- Voyis IMU: inside the camera housing. Placed at the left camera link
+       as an identity placeholder — TODO: replace with the factory extrinsics
+       (SDK ImuCalibration_t::body_T_imu, dump with SaveCalibrationDataApp),
+       including the IMU axis orientation. -->
+  <link name="voyis_imu"/>
+  <joint name="voyis_left_to_imu" type="fixed">
+    <parent link="voyis_left_link"/>
+    <child link="voyis_imu"/>
+    <origin xyz="0 0 0" rpy="0 0 0"/>
+  </joint>
 </robot>

File: urdf/rhody2.urdf.xacro (robot description, xacro)
@@ -58,6 +58,9 @@
        +/- baseline/2 in y. voyis_baseline must match the factory stereo
        calibration (SDK ExtrinsicCalibrationData_t::stereo_baseline; dump it
-       with SaveCalibrationDataApp). -->
-  <xacro:property name="voyis_baseline" value="0.160"/>
+       with SaveCalibrationDataApp).
+       Value below is the factory baseline for head 180114031, read from the
+       survey export's Voyis/Calibration_180114031/AgisoftSlaveOffsets.json
+       (x = 0.16969684810099406) and corroborated by colmap_rig.json. -->
+  <xacro:property name="voyis_baseline" value="0.16969684810099406"/>
   <xacro:property name="voyis_x" value="0.3054"/>
   <xacro:property name="voyis_z" value="0.0908"/>
@@ -69,5 +72,5 @@
     <origin xyz="${voyis_x} ${voyis_baseline/2} ${voyis_z}" rpy="0 0 0"/>
   </joint>
-  <xacro:optical_frame name="voyis_left_optical_frame" parent="voyis_left_link"/>
+  <xacro:optical_frame name="voyis_left_optical" parent="voyis_left_link"/>
   <!-- Voyis Stereo: Right Entrance Pupil (starboard side) -->
   <link name="voyis_right_link"/>
@@ -77,4 +80,14 @@
     <origin xyz="${voyis_x} ${-voyis_baseline/2} ${voyis_z}" rpy="0 0 0"/>
   </joint>
-  <xacro:optical_frame name="voyis_right_optical_frame" parent="voyis_right_link"/>
+  <xacro:optical_frame name="voyis_right_optical" parent="voyis_right_link"/>
+  <!-- Voyis IMU: inside the camera housing. Placed at the left camera link
+       as an identity placeholder — TODO: replace with the factory extrinsics
+       (SDK ImuCalibration_t::body_T_imu, dump with SaveCalibrationDataApp),
+       including the IMU axis orientation. -->
+  <link name="voyis_imu"/>
+  <joint name="voyis_left_to_imu" type="fixed">
+    <parent link="voyis_left_link"/>
+    <child link="voyis_imu"/>
+    <origin xyz="0 0 0" rpy="0 0 0"/>
+  </joint>
 </robot>
