Commit message: Add Sonardyne SPRINT-Nav Mini INS/DVL integration
Integrates the Sonardyne SPRINT-Nav Mini INS/DVL sensor, providing navigation data (IMU, DVL, depth, etc.) for the Rhody 2 platform.

This includes:
*   ROS 2 configuration for the device, specifying network parameters and topic mappings.
*   A launch file to run the `sprintnav_driver` node within the `rhody` namespace.
*   A URDF link to represent the sensor's physical presence on the robot.

File: urdf/rhody2.urdf.xacro (robot description, xacro)
@@ -38,4 +38,14 @@
     <child link="usbl_link"/>
     <origin xyz="-0.0768 0 0.3098" rpy="0 0 0"/>
+  </joint>
+  <!-- SPRINT-Nav Mini INS/DVL. TODO: measure mounting offset/orientation.
+       Note: HNAV depth is reported at the vehicle CRP configured on the
+       device web UI; HNAV altitude is at the DVL head (not attitude
+       compensated). -->
+  <link name="sprintnav_link"/>
+  <joint name="base_to_sprintnav" type="fixed">
+    <parent link="base_link"/>
+    <child link="sprintnav_link"/>
+    <origin xyz="0 0 0" rpy="0 0 0"/>
   </joint>
   <!-- FLS (Gemini): measured in Shapr3D from sonar to DVL:

Commit message: update to launches and configs and tfs for iLBL tesdt

File: urdf/rhody2.urdf.xacro (robot description, xacro)
@@ -10,4 +10,21 @@
   <xacro:arg name="fov" default="false" />
   <!-- base_link follows REP-103: x forward, y port, z up. -->
+  <!-- ==================================================================
+       base_link is the USBL.
+       Every hull offset below was measured in Shapr3D *relative to the
+       Nucleus DVL*, because base_link used to sit there (as on Rhody 1).
+       Those measurements are kept verbatim and shifted into the USBL frame
+       by the single offset below, so the numbers in the comments still match
+       the model and a re-measure of the USBL<->DVL offset only changes one
+       place.
+       Anchored to the USBL rather than the Nucleus on purpose: the Nucleus is
+       a temporary test fit, and a base_link defined by a sensor that gets
+       removed leaves every other extrinsic referred to a point that is no
+       longer on the vehicle.
+       USBL -> Nucleus DVL: dX 3.0246 in forward, dZ 12.1969 in below
+       (the USBL sits on top of the hull, aft of and above the DVL).
+       ================================================================== -->
+  <xacro:property name="usbl_to_dvl_x" value="0.0768"  scope="global"/>
+  <xacro:property name="usbl_to_dvl_z" value="-0.3098" scope="global"/>
   <!-- Base Link -->
   <link name="base_link">
@@ -23,39 +40,91 @@
     </visual>
   </link>
-  <!-- DVL Link: base_link origin is at the DVL (as on Rhody 1) -->
-  <link name="dvl_link"/>
-  <joint name="base_to_dvl" type="fixed">
-    <parent link="base_link"/>
-    <child link="dvl_link"/>
-    <origin xyz="0 0 0" rpy="0 0 0"/>
-  </joint>
-  <!-- USBL: measured in Shapr3D from USBL to DVL:
-       dX 3.0246 in, dZ 12.1969 in (0.0768, 0.3098 m). On the vehicle
-       centerline (y = 0), on top of the vehicle, aft of the DVL. -->
+  <!-- USBL (Subsonus): base_link origin is here, so translation is zero. Kept
+       as its own link so sensor data names the device rather than base_link.
+       ORIENTATION: this frame IS the device's output axes, per REP-145 - the
+       driver publishes body vectors exactly as reported. Advanced Navigation's
+       body frame is forward +X, right +Y, up -Z (Subsonus manual 9.1.3.3), i.e.
+       FRD, a 180 deg roll from base_link. The subsea unit mounts on top of the
+       vehicle pointing at the surface (7.3.2); with the web UI's Alignment
+       Configuration (9.1.3.5) set to Orientation=Subsea and the alignment
+       offsets correct, the device re-expresses its output in the VEHICLE's
+       FRD axes regardless of how the housing sits, which is what this assumes.
+       *** PROVISIONAL - confirm on the bench: *** with the vehicle level and
+       still, imu_raw.linear_acceleration.z reads about -9.8 if this frame is
+       right (z down, so gravity's reaction is -z) and about +9.8 if the
+       device is actually outputting z-up, in which case this roll is wrong.
+       Also confirm the web UI Orientation is "Subsea", not "Surface". -->
   <link name="usbl_link"/>
   <joint name="base_to_usbl" type="fixed">
     <parent link="base_link"/>
     <child link="usbl_link"/>
-    <origin xyz="-0.0768 0 0.3098" rpy="0 0 0"/>
+    <origin xyz="0 0 0" rpy="${pi} 0 0"/>
   </joint>
-  <!-- SPRINT-Nav Mini INS/DVL. TODO: measure mounting offset/orientation.
+  <!-- Nortek Nucleus 1000 DVL. Named to match what nucleus_driver_ros2
+       actually publishes (frame_id: nucleus_dvl) and the sensor_fov.yaml
+       section and meshes/fov/nucleus_dvl_*.stl, rather than the old generic
+       dvl_link - there are two DVLs on the vehicle, so "the DVL" is ambiguous.
+       Origin is the Shapr3D USBL->DVL measurement.
+       ORIENTATION: this frame IS the instrument's own axes, per REP-145 - the
+       driver publishes every topic exactly as the device reports it, and this
+       declaration is what makes that correct on the vehicle. Nortek's
+       instrument frame when mounted downward-facing (N3015-033 figure 4) is
+       x-forward, y-starboard, z-down, which is a 180 deg roll from base_link
+       (x-forward, y-port, z-up). That assumes the head is fitted with its
+       X-axis pointing forward, which Nortek recommends but does not require
+       (section 4.3). *** PROVISIONAL - confirm the mounting yaw on the
+       vehicle. *** The connector direction is the quickest tell: in figure 4
+       the connector exits along -X, i.e. aft when X points forward. -->
+  <link name="nucleus_dvl"/>
+  <joint name="base_to_nucleus" type="fixed">
+    <parent link="base_link"/>
+    <child link="nucleus_dvl"/>
+    <origin xyz="${usbl_to_dvl_x} 0 ${usbl_to_dvl_z}" rpy="${pi} 0 0"/>
+  </joint>
+  <!-- Sonardyne SPRINT-Nav Mini INS/DVL, the second DVL aboard for the
+       comparison testing.
+       *** PROVISIONAL - NOT MEASURED. *** From recollection: bottom-mounted
+       like the Nucleus, on the centerline, roughly 8 in (0.2032 m) aft of the
+       Nucleus. z is assumed equal to the Nucleus since both sit on the hull
+       bottom, and the orientation is assumed aligned with base_link. Neither
+       was measured.
+       This matters for the two-DVL comparison: the two heads are separated by
+       a lever arm r, so under rotation they legitimately measure different
+       velocities by omega x r. At 0.2 m and 10 deg/s that is ~3.5 cm/s, the
+       same order as DVL accuracy, so comparison results are only as good as
+       this number. An uncorrected mounting yaw rotates the velocity vector
+       between the two frames on top of that.
+       TODO: measure dX/dY/dZ and the mounting orientation.
        Note: HNAV depth is reported at the vehicle CRP configured on the
        device web UI; HNAV altitude is at the DVL head (not attitude
-       compensated). -->
+       compensated).
+       ORIENTATION: this frame IS the sensor's own axes, per REP-145 - the
+       driver publishes body vectors exactly as HNAV reports them, which is
+       x-forward, y-starboard, z-down (FRD), a 180 deg roll from base_link.
+       Assumes the unit is fitted DVL-face down with its forward axis along
+       the vehicle's, like the Nucleus. *** PROVISIONAL - confirm the
+       mounting yaw on the vehicle *** (same tell as the Nucleus: with the
+       vehicle still, velocity.z and the HNAV status telegram should agree
+       on sign with the Nucleus's, and a forward nudge must give +x). -->
+  <xacro:property name="sprintnav_aft_of_nucleus" value="0.2032"/>
   <link name="sprintnav_link"/>
   <joint name="base_to_sprintnav" type="fixed">
     <parent link="base_link"/>
     <child link="sprintnav_link"/>
-    <origin xyz="0 0 0" rpy="0 0 0"/>
+    <origin xyz="${usbl_to_dvl_x - sprintnav_aft_of_nucleus} 0 ${usbl_to_dvl_z}"
+            rpy="${pi} 0 0"/>
   </joint>
   <!-- FLS (Gemini): measured in Shapr3D from sonar to DVL:
        dX 14.9247 in, dY 6.0827 in, dZ 8.7819 in (0.3791, 0.1545, 0.2231 m).
        Forward of the DVL, port of centerline, above the DVL.
-       5 deg down pitch. -->
-  <link name="fls_link"/>
-  <joint name="base_to_fls" type="fixed">
+       5 deg down pitch.
+       Named to match the driver's frame_id (gemini_fls) and the
+       sensor_fov.yaml section, rather than the old fls_link. -->
+  <link name="gemini_fls"/>
+  <joint name="base_to_gemini" type="fixed">
     <parent link="base_link"/>
-    <child link="fls_link"/>
-    <origin xyz="0.3791 0.1545 0.2231" rpy="0 ${5.0 * deg} 0"/>
+    <child link="gemini_fls"/>
+    <origin xyz="${0.3791 + usbl_to_dvl_x} 0.1545 ${0.2231 + usbl_to_dvl_z}"
+            rpy="0 ${5.0 * deg} 0"/>
   </joint>
   <!-- Camera optical frame: z forward, x right, y down (REP-103 / ISAAC ROS) -->
@@ -68,5 +137,6 @@
     </joint>
   </xacro:macro>
-  <!-- Voyis Stereo: measured in Shapr3D from left camera to DVL:
+  <!-- Voyis Stereo: measured in Shapr3D from left camera to DVL (shifted
+       into the USBL frame by usbl_to_dvl_*, like the others):
        dX 12.0228 in, dZ 3.5748 in (0.3054, 0.0908 m). The stereo pair is
        centered on the vehicle centerline, so each camera sits at
@@ -85,5 +155,5 @@
     <parent link="base_link"/>
     <child link="voyis_left_link"/>
-    <origin xyz="${voyis_x} ${voyis_baseline/2} ${voyis_z}" rpy="0 0 0"/>
+    <origin xyz="${voyis_x + usbl_to_dvl_x} ${voyis_baseline/2} ${voyis_z + usbl_to_dvl_z}" rpy="0 0 0"/>
   </joint>
   <xacro:optical_frame name="voyis_left_optical" parent="voyis_left_link"/>
@@ -93,5 +163,5 @@
     <parent link="base_link"/>
     <child link="voyis_right_link"/>
-    <origin xyz="${voyis_x} ${-voyis_baseline/2} ${voyis_z}" rpy="0 0 0"/>
+    <origin xyz="${voyis_x + usbl_to_dvl_x} ${-voyis_baseline/2} ${voyis_z + usbl_to_dvl_z}" rpy="0 0 0"/>
   </joint>
   <xacro:optical_frame name="voyis_right_optical" parent="voyis_right_link"/>

File: urdf/sensor_fov.xacro (robot description, xacro)
@@ -64,5 +64,5 @@
   <!-- The 5 deg down-pitch comes from base_to_fls, not from here.        -->
   <!-- ================================================================== -->
-  <xacro:fov_volume name="fls_fov" parent="fls_link"
+  <xacro:fov_volume name="fls_fov" parent="gemini_fls"
                     mesh="gemini_fls_fan" material="fov_gemini">
     <origin xyz="0 0 0" rpy="0 0 0"/>
@@ -81,5 +81,8 @@
     <parent link="base_link"/>
     <child link="waterlinked_link"/>
-    <origin xyz="0.3791 -0.1545 0.2231" rpy="0 ${5.0 * fov_deg} 0"/>
+    <!-- Mirror of the FLS mount, so it carries the same DVL-referenced
+         measurement shifted into the USBL frame. -->
+    <origin xyz="${0.3791 + usbl_to_dvl_x} -0.1545 ${0.2231 + usbl_to_dvl_z}"
+            rpy="0 ${5.0 * fov_deg} 0"/>
   </joint>
   <xacro:fov_volume name="waterlinked_fov" parent="waterlinked_link"
@@ -97,8 +100,15 @@
   <!-- The altimeter is the theta = 0 case, so it needs no rotation.      -->
   <!--                                                                    -->
-  <!-- dvl_slant is ASSUMED at 25 deg - Nortek's published Nucleus1000    -->
-  <!-- figure, not stated in docs/N3015-033. See config/sensor_fov.yaml.  -->
+  <!-- dvl_slant is from the Nucleus 1000 datasheet (rev 03/23/2025),     -->
+  <!-- "Slanted beam angle 20 deg". Not stated in docs/N3015-033, which   -->
+  <!-- is why this was previously an assumed 25 deg.                      -->
+  <!--                                                                    -->
+  <!-- NOTE: this duplicates slant_deg in config/sensor_fov.yaml. The     -->
+  <!-- YAML drives the beam *mesh*; this property drives how the three    -->
+  <!-- beam instances are *rotated*. They must be kept in step - they     -->
+  <!-- were not, leaving the meshes at one angle and the orientations at  -->
+  <!-- another.                                                           -->
   <!-- ================================================================== -->
-  <xacro:property name="dvl_slant" value="25.0"/>
+  <xacro:property name="dvl_slant" value="20.0"/>
   <link name="dvl_fov">
     <xacro:macro name="dvl_beam" params="phi">
@@ -123,8 +133,13 @@
     </visual>
   </link>
-  <joint name="dvl_link_to_dvl_fov" type="fixed">
-    <parent link="dvl_link"/>
+  <!-- nucleus_dvl is the instrument frame (z-down, see rhody2.urdf.xacro), but
+       the beam meshes are generated opening along -z in a z-up frame. Undo
+       the instrument roll here so the drawn beams still point at the seabed.
+       Negating y maps the beam azimuths {0,120,240} onto themselves, so the
+       drawn pattern is unchanged. -->
+  <joint name="nucleus_dvl_to_dvl_fov" type="fixed">
+    <parent link="nucleus_dvl"/>
     <child link="dvl_fov"/>
-    <origin xyz="0 0 0" rpy="0 0 0"/>
+    <origin xyz="0 0 0" rpy="${pi} 0 0"/>
   </joint>
 </robot>
